File: start_wait_stop/kiCad/TimeRelay/TimeRelay.kicad_pcb (KiCad board)
At the start: 2 copper layers, 15 parts, among them J1 230V AC Input, J10 Relay, J11 Relay, J12 Relay, J13 Relay, J2 230V AC Input, J4 Relay, J5 230V AC OUTPUT, J6 230V AC OUTPUT, J9 Relay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

Commit message: Working on PCB.
Parts:
- removed J11, J12, J9: Relay, Connector_Pin:Pin_D0.9mm_L10.0mm_W2.4mm_FlatFork
- removed J5, J6: 230V AC OUTPUT, Connector_Pin:Pin_D0.9mm_L10.0mm_W2.4mm_FlatFork
- added J3: Relay NO contact, Connector_Wire:SolderWire-1.5sqmm_1x02_P7.8mm_D1.7mm_OD3.9mm, F.Cu at (101.4, 139.7)
- J1: value 230V AC Input -> 230V Input; footprint Connector_Pin:Pin_D0.9mm_L10.0mm_W2.4mm_FlatFork -> Connector_Wire:SolderWire-1.5sqmm_1x02_P7.8mm_D1.7mm_OD3.9mm
- J10: value Relay -> Relay command
- J2: value 230V AC Input -> 230V Output; footprint Connector_Pin:Pin_D0.9mm_L10.0mm_W2.4mm_FlatFork -> Connector_Wire:SolderWire-1.5sqmm_1x02_P7.8mm_D1.7mm_OD3.9mm
- J4: value Relay -> Conn_01x02_Socket; footprint Connector_Pin:Pin_D0.9mm_L10.0mm_W2.4mm_FlatFork -> Connector_Wire:SolderWire-1.5sqmm_1x02_P7.8mm_D1.7mm_OD3.9mm
- moved PS1 139.2 mm to (107.5, 120.7), turned to 180 degrees
- moved J2 125.9 mm to (91.4, 139.7), turned to 180 degrees
- moved J1 116.2 mm to (63.3, 139.7)
- moved Time1 94.8 mm to (114.6, 76.2), turned to -90 degrees
- moved J10 90.2 mm to (116.8, 97.9)
- moved A1 85.7 mm to (33.0, 83.8)
- moved SW1 62.8 mm to (93.6, 78.8)
- moved J4 43.5 mm to (64.6, 39.4), turned to -90 degrees
- moved J13 31.9 mm to (29.0, 39.4)
- moved K1 9.88 mm to (38.1, 45.7)
Connections:
- A1 pad 1: (no net) -> unconnected-(A1-TX1-Pad1)
- A1 pad 10: (no net) -> unconnected-(A1-D7-Pad10)
- A1 pad 11: (no net) -> unconnected-(A1-D8-Pad11)
- A1 pad 12: (no net) -> unconnected-(A1-D9-Pad12)
- A1 pad 13: (no net) -> unconnected-(A1-D10-Pad13)
- A1 pad 14: (no net) -> unconnected-(A1-MOSI-Pad14)
- A1 pad 15: (no net) -> unconnected-(A1-MISO-Pad15)
- A1 pad 16: (no net) -> unconnected-(A1-SCK-Pad16)
- A1 pad 17: (no net) -> unconnected-(A1-3V3-Pad17)
- A1 pad 19: (no net) -> unconnected-(A1-A0-Pad19)
- A1 pad 2: (no net) -> unconnected-(A1-RX1-Pad2)
- A1 pad 20: (no net) -> unconnected-(A1-A1-Pad20)
- A1 pad 21: (no net) -> unconnected-(A1-A2-Pad21)
- A1 pad 22: (no net) -> unconnected-(A1-A3-Pad22)
- A1 pad 23: (no net) -> unconnected-(A1-SDA/A4-Pad23)
- A1 pad 24: (no net) -> unconnected-(A1-SCL/A5-Pad24)
- A1 pad 25: (no net) -> unconnected-(A1-A6-Pad25)
- A1 pad 27: (no net) -> unconnected-(A1-+5V-Pad27)
- A1 pad 28: (no net) -> unconnected-(A1-~{RESET}-Pad28)
- A1 pad 29: Net-(J10-Pin_3) -> GND
- A1 pad 3: (no net) -> unconnected-(A1-~{RESET}-Pad3)
- A1 pad 30: (no net) -> Net-(A1-VIN)
- A1 pad 4: Net-(J10-Pin_3) -> GND
- A1 pad 5: (no net) -> Net-(A1-D2)
- A1 pad 6: (no net) -> Net-(A1-D3)
- A1 pad 7: (no net) -> unconnected-(A1-D4-Pad7)
- A1 pad 8: (no net) -> unconnected-(A1-D5-Pad8)
- A1 pad 9: (no net) -> unconnected-(A1-D6-Pad9)
- J10 pad 3: Net-(J10-Pin_3) -> GND
- J13 pad 1: (no net) -> unconnected-(J13-Pin_1-Pad1)
- J4 pad 1: (no net) -> Net-(J4-Pin_1)
- K1 pad 11: (no net) -> Net-(J4-Pin_1)
- K1 pad 12: (no net) -> unconnected-(K1-Pad12)
- K1 pad 14: (no net) -> Net-(J4-Pin_2)
- K1 pad A1: (no net) -> Net-(J13-Pin_3)
- K1 pad A2: (no net) -> Net-(J13-Pin_2)
- PS1 pad 1: (no net) -> Net-(J1-Pin_1)
- PS1 pad 2: (no net) -> Net-(J1-Pin_2)
- PS1 pad 3: Net-(J10-Pin_3) -> GND
- SW1 pad 1: Net-(J10-Pin_3) -> GND
- Time1 pad 1: (no net) -> Net-(A1-AREF)
- Time1 pad 2: (no net) -> Net-(A1-A7)
- Time1 pad 3: (no net) -> GND
Routing:
- net GND: track 0.00 -> 195.7 mm, vias 0 -> 4
- net Net-(A1-D2): track 0.00 -> 135.3 mm, vias 0 -> 2
- net Net-(A1-VIN): track 0.00 -> 122.0 mm, vias 0 -> 3
- net Net-(A1-AREF): track 0.00 -> 110.8 mm
- net Net-(J1-Pin_2): track 0.00 -> 101.4 mm
- net Net-(A1-D3): track 0.00 -> 92.2 mm
- net Net-(A1-A7): track 0.00 -> 77.1 mm
- net Net-(J1-Pin_1): track 0.00 -> 65.8 mm
- net Net-(J2-Pin_1): track 0.00 -> 9.98 mm
Other:
- board outline added: 99.1 x 73.7 mm
